File: Oven_hw/Oven.kicad_pcb (KiCad board)
At the start: 2 copper layers, 87 x 50 mm, 100 parts, among them Q1 NSS20101, SW1 BUTTON6x6, U1 ER-TFT024

Commit message: + PCB sent to factory
Parts:
- removed XL7: CONN_4, Connectors:PLS-4
- C1, C10, C13, C14, C15, C16, C2, C25, C28, C3, C31, C34, C4, C42, C5, C6, C7, C9, DA1, DA2, DD2, F1, F2, L1, L2, R1, R14, R15, R17, R18, R19, R2, R20, R22, R3, R5, R6, R7, R8: moved to B.Cu
- R4: value 10k 0.1% -> 10k0.1%; moved to B.Cu
- moved R15 79.5 mm to (149.2, 88.2), turned to 90 degrees
- moved R14 79.3 mm to (151.0, 88.2), turned to 270 degrees
- moved R17 76.6 mm to (134.6, 122.0)
- moved R3 75.1 mm to (149.4, 126.2)
- moved C31 73.5 mm to (134.0, 101.8)
- moved C28 72.4 mm to (134.0, 100.2)
- moved C25 70.7 mm to (153.2, 88.2), turned to 90 degrees
- moved C34 69.3 mm to (134.0, 98.6)
- moved F2 67.8 mm to (147.0, 115.2), turned to 90 degrees
- moved DA2 67.4 mm to (151.8, 130.0), turned to 270 degrees
- moved R18 66.5 mm to (134.6, 120.4)
- moved R19 63.3 mm to (134.6, 118.8)
- moved C16 61.2 mm to (147.0, 126.2), turned to 90 degrees
- moved R20 60.5 mm to (134.6, 117.2)
- moved R5 59.5 mm to (159.6, 120.8), turned to 180 degrees
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Connections:
- C42 pad 1: GND -> GNDPWR
- DD1 pad 20: Net-(DD1-Pad20) -> (no net)
- DD1 pad 39: /LCD_RST -> (no net)
- DD1 pad 40: /LCD_DC -> (no net)
- DD1 pad 41: Net-(DD1-Pad41) -> (no net)
- DD1 pad 42: Net-(DD1-Pad42) -> (no net)
- DD1 pad 50: (no net) -> /LCD_DC
- DD1 pad 54: (no net) -> /LCD_RST
- R1 pad 1: +3.3V_A -> /ADC_PWR1
- R16 pad 1: Net-(DD1-Pad42) -> Net-(DD1-Pad15)
- R22 pad 2: GND -> GNDPWR
- R3 pad 1: +3.3V_A -> /ADC_PWR2
Routing:
- net GND: track 0.00 -> 569.8 mm, vias 0 -> 91
- net /SHLD: track 0.00 -> 167.3 mm
- net AGND: track 0.00 -> 160.8 mm, vias 0 -> 31
- net GNDPWR: track 0.00 -> 120.1 mm, vias 0 -> 2
- net PwrMCU: track 0.00 -> 116.7 mm, vias 0 -> 9
- net +12V: track 0.00 -> 104.9 mm, vias 0 -> 2
- net +3.3V: track 0.00 -> 98.6 mm, vias 0 -> 5
- net +5V: track 0.00 -> 57.4 mm, vias 0 -> 2
- net Net-(R23-Pad2): track 0.00 -> 47.2 mm, vias 0 -> 1
- net Net-(DD1-Pad60): track 0.00 -> 45.0 mm, vias 0 -> 4
- net /VENT_CTRL: track 0.00 -> 44.2 mm, vias 0 -> 2
- net /HEATER_CTRL: track 0.00 -> 43.5 mm, vias 0 -> 2
- net /D+: track 0.00 -> 39.1 mm, vias 0 -> 1
- net /SCL: track 0.00 -> 37.9 mm, vias 0 -> 3
- net /UART_RX: track 0.00 -> 36.8 mm, vias 0 -> 2
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- added copper zone on B.Cu, net AGND
- added copper zone on F.Cu, net AGND
- added copper zone on B.Cu, net GND
- added copper zone on F.Cu, net GND
Other:
- board size 87 x 50 mm -> 89 x 50 mm
- net class Default: trace_width 0.25 -> 0.2; via_dia 0.6 -> 0.7; via_drill 0.4 -> 0.3
- net class Wide added: clearance 0.2, trace_width 0.5, via_dia 0.9, via_drill 0.4
- rule pad_to_mask_clearance: 0.2 -> 0.1
- board text added: "EE"
- board text added: "Fan"
- board text added: "Heater"
- board text added: "Oven v1"
- board text added: "Sns Heater"
- board text added: "Sns PCB"
- board text added: "Touch"
